File: FSAE Main Panel/Display.sch (KiCad schematic (older format))
At the start: 66 parts, among them U501 TLC6C598, U502 TLC6C5816, U503 TLC6C5816, U504 TLC6C5816

Commit message: Updated to KiCad 5
Parts:
- C501, C502: symbol C -> Device:C
- C503, C504, C505, C506: renamed from C?; symbol C -> Device:C
- D501: symbol SA10-11GWA -> KingBright_Addition:SA10-11GWA
- D502, D503, D504, D505, D506, D507, D508, D509, D510, D511, D512, D513, D514, D515, D516, D517, D518, D519, D520, D521, D522, D523, D524, D525, D526, D527, D528, D529, D530, D531, D532, D533, D534, D535, D536, D537, D538, D539, D540, D541, D542, D543, D544, D545, D546, D547, D548, D549: symbol LED_Small -> Device:LED_Small
- RN501, RN502, RN503, RN504, RN505, RN506, RN507: symbol R_Pack08 -> Device:R_Pack08
- U501: symbol TLC6C598 -> TI_Additions:TLC6C598
- U502, U503, U504: symbol TLC6C5816 -> TI_Additions:TLC6C5816
Connections:
- wire segments 480 -> 414

Commit message: Updated Footprint Association
Parts:
- C501: footprint (none) -> Capacitors_SMD:C_1206; Description (none) -> Ceramic 1uF 25V X7R 1206
- C502, C504, C505, C506: footprint (none) -> Capacitors_SMD:C_1206; Description (none) -> Ceramic 0.1uF 10V X7R 1206
- C503: footprint (none) -> Capacitors_SMD:C_1206; Description (none) -> Ceramic 4.7uF 10V X5R 1206
Changed lines of the file:
@@
 F 0 "C502" H 1975 6600 50  0000 L CNN
 F 1 "100nF" H 1975 6400 50  0000 L CNN
-F 2 "" H 1988 6350 50  0001 C CNN
+F 2 "Capacitors_SMD:C_1206" H 1988 6350 50  0001 C CNN
 F 3 "" H 1950 6500 50  0001 C CNN
+F 4 "Ceramic 0.1uF 10V X7R 1206" H 1950 6500 50  0001 C CNN "Description"
 	1    1950 6500
 	1    0    0    -1
@@
 F 0 "C501" H 1725 6600 50  0000 L CNN
 F 1 "1uF" H 1725 6400 50  0000 L CNN
-F 2 "" H 1738 6350 50  0001 C CNN
+F 2 "Capacitors_SMD:C_1206" H 1738 6350 50  0001 C CNN
 F 3 "" H 1700 6500 50  0001 C CNN
+F 4 "Ceramic 1uF 25V X7R 1206" H 1700 6500 50  0001 C CNN "Description"
 	1    1700 6500
 	1    0    0    -1
@@
 F 0 "C504" H 2575 3300 50  0000 L CNN
 F 1 "100nF" H 2575 3100 50  0000 L CNN
-F 2 "" H 2588 3050 50  0001 C CNN
+F 2 "Capacitors_SMD:C_1206" H 2588 3050 50  0001 C CNN
 F 3 "" H 2550 3200 50  0001 C CNN
+F 4 "Ceramic 0.1uF 10V X7R 1206" H 2550 3200 50  0001 C CNN "Description"
 	1    2550 3200
 	-1   0    0    1
@@
 F 0 "C503" H 1225 3300 50  0000 L CNN
 F 1 "4.7uF" H 1225 3100 50  0000 L CNN
-F 2 "" H 1238 3050 50  0001 C CNN
+F 2 "Capacitors_SMD:C_1206" H 1238 3050 50  0001 C CNN
 F 3 "" H 1200 3200 50  0001 C CNN
+F 4 "Ceramic 4.7uF 10V X5R 1206" H 1200 3200 50  0001 C CNN "Description"
 	1    1200 3200
 	-1   0    0    1
@@
 F 0 "C505" H 4275 3300 50  0000 L CNN
 F 1 "100nF" H 4275 3100 50  0000 L CNN
-F 2 "" H 4288 3050 50  0001 C CNN
+F 2 "Capacitors_SMD:C_1206" H 4288 3050 50  0001 C CNN
 F 3 "" H 4250 3200 50  0001 C CNN
+F 4 "Ceramic 0.1uF 10V X7R 1206" H 4250 3200 50  0001 C CNN "Description"
 	1    4250 3200
 	-1   0    0    1
@@
 F 0 "C506" H 5975 3300 50  0000 L CNN
 F 1 "100nF" H 5975 3100 50  0000 L CNN
-F 2 "" H 5988 3050 50  0001 C CNN
+F 2 "Capacitors_SMD:C_1206" H 5988 3050 50  0001 C CNN
 F 3 "" H 5950 3200 50  0001 C CNN
+F 4 "Ceramic 0.1uF 10V X7R 1206" H 5950 3200 50  0001 C CNN "Description"
 	1    5950 3200
 	-1   0    0    1
 $EndComp
 $Comp
-L power:+3.3V #PWR501
+L power:+3.3V #PWR0501
 U 1 1 5BEAB3A4
 P 800 3000
-F 0 "#PWR501" H 800 2850 50  0001 C CNN
+F 0 "#PWR0501" H 800 2850 50  0001 C CNN
 F 1 "+3.3V" H 800 3140 50  0000 C CNN
 F 2 "" H 800 3000 50  0001 C CNN
@@
 $EndComp
 $Comp
-L power:GND #PWR503
+L power:GND #PWR0503
 U 1 1 5BEAB544
 P 1200 3450
-F 0 "#PWR503" H 1200 3200 50  0001 C CNN
+F 0 "#PWR0503" H 1200 3200 50  0001 C CNN
 F 1 "GND" H 1200 3300 50  0000 C CNN
 F 2 "" H 1200 3450 50  0001 C CNN
@@
 $EndComp
 $Comp
-L power:GND #PWR505
+L power:GND #PWR0505
 U 1 1 5BEAB5DA
 P 2700 3500
-F 0 "#PWR505" H 2700 3250 50  0001 C CNN
+F 0 "#PWR0505" H 2700 3250 50  0001 C CNN
 F 1 "GND" H 2700 3350 50  0000 C CNN
 F 2 "" H 2700 3500 50  0001 C CNN
@@
 $EndComp
 $Comp
-L power:GND #PWR506
+L power:GND #PWR0506
 U 1 1 5BEAB669
 P 4400 3500
-F 0 "#PWR506" H 4400 3250 50  0001 C CNN
+F 0 "#PWR0506" H 4400 3250 50  0001 C CNN
 F 1 "GND" H 4400 3350 50  0000 C CNN
 F 2 "" H 4400 3500 50  0001 C CNN
@@
 $EndComp
 $Comp
-L power:GND #PWR507
+L power:GND #PWR0507
 U 1 1 5BEAB7A8
 P 6100 3500
-F 0 "#PWR507" H 6100 3250 50  0001 C CNN
+F 0 "#PWR0507" H 6100 3250 50  0001 C CNN
 F 1 "GND" H 6100 3350 50  0000 C CNN
 F 2 "" H 6100 3500 50  0001 C CNN
@@
 RPM_OUT
 $Comp
-L power:+3.3V #PWR504
+L power:+3.3V #PWR0504
 U 1 1 5BEAF345
 P 1200 6250
-F 0 "#PWR504" H 1200 6100 50  0001 C CNN
+F 0 "#PWR0504" H 1200 6100 50  0001 C CNN
 F 1 "+3.3V" H 1200 6390 50  0000 C CNN
 F 2 "" H 1200 6250 50  0001 C CNN
@@
 LED_5V+
 $Comp
-L power:GND #PWR502
+L power:GND #PWR0502
 U 1 1 5BEAF6F1
 P 900 7450
-F 0 "#PWR502" H 900 7200 50  0001 C CNN
+F 0 "#PWR0502" H 900 7200 50  0001 C CNN
 F 1 "GND" H 900 7300 50  0000 C CNN
 F 2 "" H 900 7450 50  0001 C CNN
@@
 	5750 6300 5850 6300
 Wire Wire Line
-	5850 6300 5850 6500
+	5850 6300 5850 6400
 Wire Wire Line
 	5850 6500 5750 6500
 Wire Wire Line
-	5750 6400 6000 6400
+	5750 6400 5850 6400
 Connection ~ 5850 6400
 Wire Wire Line
@@
 	2450 6350 2550 6350
 Wire Wire Line
-	900  7450 3700 7450
+	900  7450 1700 7450
 Wire Wire Line
 	6000 6400 6000 6050
@@
 	2450 6250 2450 6350
 Wire Wire Line
-	1200 6250 2450 6250
+	1200 6250 1700 6250
 Wire Wire Line
 	1700 6350 1700 6250
@@
 	10500 1200 10500 1800
 Wire Wire Line
-	5250 900  10950 900
+	5250 900  6000 900
 Wire Wire Line
 	10500 900  10500 1000
@@
 Wire Wire Line
 	1450 3800 1300 3800
-Wire Bus Line
-	1200 3900 1200 5000
 Wire Wire Line
 	4250 3800 4450 3800
@@
 Wire Wire Line
 	4850 3800 4650 3800
-Wire Bus Line
-	6250 3900 6250 5000
-Wire Bus Line
-	2850 3900 2850 5000
-Wire Bus Line
-	4550 3900 4550 5000
 Connection ~ 10200 900
 Wire Wire Line
 	5950 3000 5950 3050
 Wire Wire Line
-	800  3000 5950 3000
+	800  3000 1200 3000
 Wire Wire Line
 	4250 3000 4250 3050
@@
 	1350 4700 1350 5300
 Wire Wire Line
-	1000 5200 4800 5200
+	1000 5200 1400 5200
 Connection ~ 1400 5200
 Wire Wire Line
-	1000 5300 4750 5300
+	1000 5300 1350 5300
 Connection ~ 1350 5300
 Connection ~ 3050 5300
@@
 Wire Wire Line
 	10950 2500 10950 2650
-Wire Bus Line
-	6450 2750 11100 2750
 Wire Wire Line
 	8500 4000 8550 4000
@@
 	10300 3250 10300 3100
 Wire Wire Line
-	8400 4600 10750 4600
+	8400 4600 8550 4600
 Wire Wire Line
 	8400 4600 8400 4500
@@
 Wire Bus Line
 	4700 2900 1250 2900
-Wire Bus Line
-	1300 2900 1300 3600
 Text GLabel 1250 2900 0    39   Input ~ 0
 RPM_PWM
-Wire Bus Line
-	4700 2900 4700 3600
-Wire Bus Line
-	3000 2900 3000 3600
 Wire Wire Line
 	4850 3600 4800 3600
@@
 Text Label 4800 3700 0    39   ~ 0
 ~G6
-Wire Bus Line
-	1300 5100 6600 5100
-Wire Bus Line
-	6600 3000 11100 3000
 Wire Bus Line
 	11100 3000 11100 2750
@@
 	2650 4700 2650 5400
 Wire Wire Line
-	1000 5400 6050 5400
+	1000 5400 2650 5400
 Wire Wire Line
 	4350 4700 4350 5400
@@
 	6100 5500 6100 4600
 Wire Wire Line
-	1000 5500 6100 5500
+	1000 5500 2700 5500
 Wire Wire Line
 	4400 4600 4400 5500
@@
 Text Label 2500 7050 0    39   ~ 0
 ~G7
+Wire Wire Line
+	5850 6400 5850 6500
+Wire Wire Line
+	5850 6400 6000 6400
+Wire Wire Line
+	1700 6250 1950 6250
+Wire Wire Line
+	1950 6250 2450 6250
+Wire Wire Line
+	1700 7450 1950 7450
+Wire Wire Line
+	1950 7450 3700 7450
+Wire Wire Line
+	10050 900  10200 900
+Wire Wire Line
+	9900 900  10050 900
+Wire Wire Line
+	9600 900  9900 900
+Wire Wire Line
+	9450 900  9600 900
+Wire Wire Line
+	9300 900  9450 900
+Wire Wire Line
+	9150 900  9300 900
+Wire Wire Line
+	9000 900  9150 900
+Wire Wire Line
+	8850 900  9000 900
+Wire Wire Line
+	8700 900  8850 900
+Wire Wire Line
+	8550 900  8700 900
+Wire Wire Line
+	8250 900  8550 900
+Wire Wire Line
+	8100 900  8250 900
+Wire Wire Line
+	7950 900  8100 900
+Wire Wire Line
+	7800 900  7950 900
+Wire Wire Line
+	7650 900  7800 900
+Wire Wire Line
+	7500 900  7650 900
+Wire Wire Line
+	7350 900  7500 900
+Wire Wire Line
+	7200 900  7350 900
+Wire Wire Line
+	7050 900  7200 900
+Wire Wire Line
+	6900 900  7050 900
+Wire Wire Line
+	6750 900  6900 900
+Wire Wire Line
+	6600 900  6750 900
+Wire Wire Line
+	6450 900  6600 900
+Wire Wire Line
+	6300 900  6450 900
+Wire Wire Line
+	6150 900  6300 900
+Wire Wire Line
+	6000 900  6150 900
+Wire Wire Line
+	10350 900  10500 900
+Wire Wire Line
+	10200 900  10350 900
+Wire Wire Line
+	4250 3000 4800 3000
+Wire Wire Line
+	3100 3000 4250 3000
+Wire Wire Line
+	4800 3000 5950 3000
+Wire Wire Line
+	2550 3000 3100 3000
+Wire Wire Line
+	1400 3000 2550 3000
+Wire Wire Line
+	1200 3000 1400 3000
+Wire Wire Line
+	1400 5200 3100 5200
+Wire Wire Line
+	1350 5300 3050 5300
+Wire Wire Line
+	3050 5300 4750 5300
+Wire Wire Line
+	3100 5200 4800 5200
+Wire Wire Line
+	10500 900  10650 900
+Wire Wire Line
+	8550 4600 8700 4600
+Wire Wire Line
+	8700 4600 8850 4600
+Wire Wire Line
+	8850 4600 9000 4600
+Wire Wire Line
+	9000 4600 9150 4600
+Wire Wire Line
+	9150 4600 9300 4600
+Wire Wire Line
+	9300 4600 9450 4600
+Wire Wire Line
+	9450 4600 9600 4600
+Wire Wire Line
+	9600 4600 9750 4600
+Wire Wire Line
+	9750 4600 9900 4600
+Wire Wire Line
+	9900 4600 10050 4600
+Wire Wire Line
+	10050 4600 10200 4600
+Wire Wire Line
+	10200 4600 10350 4600
+Wire Wire Line
+	10350 4600 10500 4600
+Wire Wire Line
+	10500 4600 10650 4600
+Wire Wire Line
+	10650 4600 10750 4600
+Wire Wire Line
+	10650 900  10800 900
+Wire Wire Line
+	10800 900  10950 900
+Wire Wire Line
+	2650 5400 4350 5400
+Wire Wire Line
+	4350 5400 6050 5400
+Wire Wire Line
+	4400 5500 6100 5500
+Wire Wire Line
+	2700 5500 4400 5500
+Wire Bus Line
+	1300 2900 1300 3600
+Wire Bus Line
+	4700 2900 4700 3600
+Wire Bus Line
+	3000 2900 3000 3600
+Wire Bus Line
+	1300 5100 6600 5100
+Wire Bus Line
+	1200 3900 1200 5000
+Wire Bus Line
+	6250 3900 6250 5000
+Wire Bus Line
+	2850 3900 2850 5000
+Wire Bus Line
+	4550 3900 4550 5000
+Wire Bus Line
+	6600 3000 11100 3000
+Wire Bus Line
+	6450 2750 11100 2750
 $EndSCHEMATC

Commit message: New footprints, finished associating footprints
Parts:
- U502, U503, U504: footprint (none) -> TLC6C5816:TLC6C5816
Changed lines of the file:
@@
 F 0 "U502" H 2000 5100 60  0000 C CNN
 F 1 "TLC6C5816" H 2000 3450 60  0000 C CNN
-F 2 "" H 2050 3500 60  0001 C CNN
+F 2 "TLC6C5816:TLC6C5816" H 2050 3500 60  0001 C CNN
 F 3 "" H 2050 3500 60  0001 C CNN
 	1    2000 4200
@@
 F 0 "U503" H 3700 5100 60  0000 C CNN
 F 1 "TLC6C5816" H 3700 3450 60  0000 C CNN
-F 2 "" H 3750 3500 60  0001 C CNN
+F 2 "TLC6C5816:TLC6C5816" H 3750 3500 60  0001 C CNN
 F 3 "" H 3750 3500 60  0001 C CNN
 	1    3700 4200
@@
 F 0 "U504" H 5400 5100 60  0000 C CNN
 F 1 "TLC6C5816" H 5400 3450 60  0000 C CNN
-F 2 "" H 5450 3500 60  0001 C CNN
+F 2 "TLC6C5816:TLC6C5816" H 5450 3500 60  0001 C CNN
 F 3 "" H 5450 3500 60  0001 C CNN
 	1    5400 4200

Commit message: Edited footprints, started PCB layout
Parts:
- RN501: footprint Housings_SOIC:SOIC-16W_5.3x10.2mm_Pitch1.27mm -> Housings_SOIC:SOIC-16_3.9x9.9mm_Pitch1.27mm
- RN502, RN503, RN504, RN505, RN506, RN507: footprint Housings_SOIC:SOIC-16W_5.3x10.2mm_Pitch1.27mm -> Bourns 4800P:Bourns 4800P SOM-16
Changed lines of the file:
@@
 F 0 "RN501" V 3900 6700 50  0000 C CNN
 F 1 "51 Ohm (8x)" V 4800 6700 50  0000 C CNN
-F 2 "Housings_SOIC:SOIC-16W_5.3x10.2mm_Pitch1.27mm" V 4875 6700 50  0001 C CNN
+F 2 "Housings_SOIC:SOIC-16_3.9x9.9mm_Pitch1.27mm" V 4875 6700 50  0001 C CNN
 F 3 "https://www.mouser.com/datasheet/2/54/800P-777115.pdf" H 4400 6700 50  0001 C CNN
 F 4 "4816P-1-510LF" V 4400 6700 60  0001 C CNN "Part Number"
@@
 F 0 "RN502" V 6250 2300 50  0000 C CNN
 F 1 "151 Ohm (8x)" V 7150 2300 50  0000 C CNN
-F 2 "Housings_SOIC:SOIC-16W_5.3x10.2mm_Pitch1.27mm" V 7225 2300 50  0001 C CNN
+F 2 "Bourns 4800P:Bourns 4800P SOM-16" V 7225 2300 50  0001 C CNN
 F 3 "https://www.mouser.com/datasheet/2/54/800P-777115.pdf" H 6750 2300 50  0001 C CNN
 F 4 "4816P-1-151" V 6750 2300 60  0001 C CNN "Part Number"
@@
 F 0 "RN503" V 7450 2300 50  0000 C CNN
 F 1 "151 Ohm (8x)" V 8350 2300 50  0000 C CNN
-F 2 "Housings_SOIC:SOIC-16W_5.3x10.2mm_Pitch1.27mm" V 8425 2300 50  0001 C CNN
+F 2 "Bourns 4800P:Bourns 4800P SOM-16" V 8425 2300 50  0001 C CNN
 F 3 "https://www.mouser.com/datasheet/2/54/800P-777115.pdf" H 7950 2300 50  0001 C CNN
 F 4 "4816P-1-151" V 7950 2300 60  0001 C CNN "Part Number"
@@
 F 0 "RN504" V 8800 2300 50  0000 C CNN
 F 1 "220 Ohm (8x)" V 9700 2300 50  0000 C CNN
-F 2 "Housings_SOIC:SOIC-16W_5.3x10.2mm_Pitch1.27mm" V 9775 2300 50  0001 C CNN
+F 2 "Bourns 4800P:Bourns 4800P SOM-16" V 9775 2300 50  0001 C CNN
 F 3 "https://www.mouser.com/datasheet/2/54/800P-777115.pdf" H 9300 2300 50  0001 C CNN
 F 4 "4816P-1-221LF" V 9300 2300 60  0001 C CNN "Part Number"
@@
 F 0 "RN505" V 10150 2300 50  0000 C CNN
 F 1 "180 Ohm (8x)" V 11050 2300 50  0000 C CNN
-F 2 "Housings_SOIC:SOIC-16W_5.3x10.2mm_Pitch1.27mm" V 11125 2300 50  0001 C CNN
+F 2 "Bourns 4800P:Bourns 4800P SOM-16" V 11125 2300 50  0001 C CNN
 F 3 "https://www.mouser.com/datasheet/2/54/800P-777115.pdf" H 10650 2300 50  0001 C CNN
 F 4 "4816P-1-181LF" V 10650 2300 60  0001 C CNN "Part Number"
@@
 F 0 "RN506" V 8300 3450 50  0000 C CNN
 F 1 "68 Ohm (8x)" V 9200 3450 50  0000 C CNN
-F 2 "Housings_SOIC:SOIC-16W_5.3x10.2mm_Pitch1.27mm" V 9275 3450 50  0001 C CNN
+F 2 "Bourns 4800P:Bourns 4800P SOM-16" V 9275 3450 50  0001 C CNN
 F 3 "https://www.mouser.com/datasheet/2/54/800P-777115.pdf" H 8800 3450 50  0001 C CNN
 F 4 "4816P-1-680LF" V 8800 3450 60  0001 C CNN "Part Number"
@@
 F 0 "RN507" V 9500 3450 50  0000 C CNN
 F 1 "68 Ohm (8x)" V 10400 3450 50  0000 C CNN
-F 2 "Housings_SOIC:SOIC-16W_5.3x10.2mm_Pitch1.27mm" V 10475 3450 50  0001 C CNN
+F 2 "Bourns 4800P:Bourns 4800P SOM-16" V 10475 3450 50  0001 C CNN
 F 3 "https://www.mouser.com/datasheet/2/54/800P-777115.pdf" H 10000 3450 50  0001 C CNN
 F 4 "4816P-1-680LF" V 10000 3450 60  0001 C CNN "Part Number"
