File: FSAE Main Panel/ExternalInterface.sch (KiCad schematic (older format))
At the start: 16 parts, among them J1 Conn_01x04, J2 TE_84953-6_FPC, J201 Conn_01x06, SW1 B3W-1020, SW2 B3W-1020

Commit message: Cortex debugger, GPIO pinning, minor fixes
Parts:
- added J?: Cortex_Debug, symbol Cortex_Debug
Connections:
- net labels added: SWCLK, SWDIO
- wire segments 49 -> 72
Changed lines of the file:
@@
 LIBS:samd21g18a-au
 LIBS:zldo1117-5v
+LIBS:cortex_debug
 LIBS:FSAE Main Panel-cache
 EELAYER 25 0
@@
 	750  3250 750  3400
 Wire Wire Line
-	1600 3250 1800 3250
-Wire Wire Line
-	2100 3250 2300 3250
-Wire Wire Line
-	1700 3050 1700 3450
+	1600 3250 1700 3250
+Wire Wire Line
+	1700 3250 1800 3250
+Wire Wire Line
+	2100 3250 2150 3250
+Wire Wire Line
+	2150 3250 2300 3250
+Wire Wire Line
+	1700 3050 1700 3250
+Wire Wire Line
+	1700 3250 1700 3450
 Connection ~ 1700 3250
 Wire Notes Line
@@
 Connection ~ 2150 3250
 Wire Wire Line
-	1600 4150 1800 4150
-Wire Wire Line
-	2100 4150 2300 4150
-Wire Wire Line
-	1700 3950 1700 4350
+	1600 4150 1700 4150
+Wire Wire Line
+	1700 4150 1800 4150
+Wire Wire Line
+	2100 4150 2150 4150
+Wire Wire Line
+	2150 4150 2300 4150
+Wire Wire Line
+	1700 3950 1700 4150
+Wire Wire Line
+	1700 4150 1700 4350
 Connection ~ 1700 4150
 Wire Notes Line
@@
 Connection ~ 2150 4150
 Wire Wire Line
-	3400 1950 5050 1950
+	3400 1950 3600 1950
+Wire Wire Line
+	3600 1950 4450 1950
+Wire Wire Line
+	4450 1950 5050 1950
 Wire Wire Line
 	3400 2350 4000 2350
 Wire Wire Line
-	4000 2350 4000 2800
-Wire Wire Line
-	3400 2050 6250 2050
+	4000 2350 4000 2750
+Wire Wire Line
+	4000 2750 4000 2800
+Wire Wire Line
+	3400 2050 4800 2050
+Wire Wire Line
+	4800 2050 6250 2050
 Wire Wire Line
 	3750 1600 3750 2150
 Connection ~ 3750 2150
 Wire Wire Line
-	3400 2150 6250 2150
+	3400 2150 3750 2150
+Wire Wire Line
+	3750 2150 6250 2150
 Wire Wire Line
 	3750 1200 3600 1200
@@
 	5600 2750 5600 2650
 Wire Wire Line
-	3400 2750 5600 2750
+	3400 2750 4000 2750
+Wire Wire Line
+	4000 2750 4450 2750
+Wire Wire Line
+	4450 2750 4900 2750
+Wire Wire Line
+	4900 2750 5600 2750
 Connection ~ 4000 2750
 Connection ~ 4900 2750
@@
 $EndComp
 Wire Wire Line
-	5350 1950 5800 1950
+	5350 1950 5600 1950
+Wire Wire Line
+	5600 1950 5800 1950
 Wire Wire Line
 	6100 1950 6250 1950
+$Comp
+L Cortex_Debug J?
+U 1 1 5BFE970B
+P 3950 3750
+F 0 "J?" H 3950 4050 50  0000 C CNN
+F 1 "Cortex_Debug" H 3950 3450 50  0000 C CNN
+F 2 "" H 4100 3750 39  0001 C CNN
+F 3 "" H 4100 3750 39  0001 C CNN
+	1    3950 3750
+	1    0    0    -1
+$EndComp
+$Comp
+L +3.3V #PWR?
+U 1 1 5BFE98A3
+P 3200 3400
+F 0 "#PWR?" H 3200 3250 50  0001 C CNN
+F 1 "+3.3V" H 3200 3540 50  0000 C CNN
+F 2 "" H 3200 3400 50  0001 C CNN
+F 3 "" H 3200 3400 50  0001 C CNN
+	1    3200 3400
+	1    0    0    -1
+$EndComp
+$Comp
+L GND #PWR?
+U 1 1 5BFE993E
+P 3200 4000
+F 0 "#PWR?" H 3200 3750 50  0001 C CNN
+F 1 "GND" H 3200 3850 50  0000 C CNN
+F 2 "" H 3200 4000 50  0001 C CNN
+F 3 "" H 3200 4000 50  0001 C CNN
+	1    3200 4000
+	1    0    0    -1
+$EndComp
+Wire Wire Line
+	3350 3550 3200 3550
+Wire Wire Line
+	3200 3550 3200 3400
+Wire Wire Line
+	3350 3650 3200 3650
+Wire Wire Line
+	3200 3650 3200 3750
+Wire Wire Line
+	3200 3750 3200 4000
+Wire Wire Line
+	3350 3750 3200 3750
+Connection ~ 3200 3750
+Text GLabel 4650 3550 2    39   Input ~ 0
+SWDIO
+Text GLabel 4650 3650 2    39   Input ~ 0
+SWCLK
+Wire Wire Line
+	4650 3550 4550 3550
+Wire Wire Line
+	4650 3650 4550 3650
+Wire Notes Line
+	3000 3200 3000 4200
+Wire Notes Line
+	3000 4200 5000 4200
+Wire Notes Line
+	5000 4200 5000 3200
+Wire Notes Line
+	5000 3200 3000 3200
 $EndSCHEMATC

Commit message: Added power regulator for LEDs, further GPIO considerations
Connections:
- net labels added: DWC_+5V
- wire segments 72 -> 56
Other:
- note added: "Cortex Debugger"
Changed lines of the file:
@@
 ~CHECK_ENGINE
 Text GLabel 1900 2050 2    39   Input ~ 0
-DWC_5V+
+DWC_+5V
 $Comp
 L GND #PWR204
@@
 	750  3250 750  3400
 Wire Wire Line
-	1600 3250 1700 3250
-Wire Wire Line
-	1700 3250 1800 3250
-Wire Wire Line
-	2100 3250 2150 3250
-Wire Wire Line
-	2150 3250 2300 3250
-Wire Wire Line
-	1700 3050 1700 3250
-Wire Wire Line
-	1700 3250 1700 3450
+	1600 3250 1800 3250
+Wire Wire Line
+	2100 3250 2300 3250
+Wire Wire Line
+	1700 3050 1700 3450
 Connection ~ 1700 3250
 Wire Notes Line
@@
 Connection ~ 2150 3250
 Wire Wire Line
-	1600 4150 1700 4150
-Wire Wire Line
-	1700 4150 1800 4150
-Wire Wire Line
-	2100 4150 2150 4150
-Wire Wire Line
-	2150 4150 2300 4150
-Wire Wire Line
-	1700 3950 1700 4150
-Wire Wire Line
-	1700 4150 1700 4350
+	1600 4150 1800 4150
+Wire Wire Line
+	2100 4150 2300 4150
+Wire Wire Line
+	1700 3950 1700 4350
 Connection ~ 1700 4150
 Wire Notes Line
@@
 Connection ~ 2150 4150
 Wire Wire Line
-	3400 1950 3600 1950
-Wire Wire Line
-	3600 1950 4450 1950
-Wire Wire Line
-	4450 1950 5050 1950
+	3400 1950 5050 1950
 Wire Wire Line
 	3400 2350 4000 2350
 Wire Wire Line
-	4000 2350 4000 2750
-Wire Wire Line
-	4000 2750 4000 2800
-Wire Wire Line
-	3400 2050 4800 2050
-Wire Wire Line
-	4800 2050 6250 2050
+	4000 2350 4000 2800
+Wire Wire Line
+	3400 2050 6250 2050
 Wire Wire Line
 	3750 1600 3750 2150
 Connection ~ 3750 2150
 Wire Wire Line
-	3400 2150 3750 2150
-Wire Wire Line
-	3750 2150 6250 2150
+	3400 2150 6250 2150
 Wire Wire Line
 	3750 1200 3600 1200
@@
 	4800 1200 4900 1200
 Wire Wire Line
-	4900 1200 4900 2750
+	4900 2750 4900 1200
 Wire Wire Line
 	5600 2750 5600 2650
 Wire Wire Line
-	3400 2750 4000 2750
-Wire Wire Line
-	4000 2750 4450 2750
-Wire Wire Line
-	4450 2750 4900 2750
-Wire Wire Line
-	4900 2750 5600 2750
+	3400 2750 5600 2750
 Connection ~ 4000 2750
 Connection ~ 4900 2750
@@
 $EndComp
 Wire Wire Line
-	5350 1950 5600 1950
-Wire Wire Line
-	5600 1950 5800 1950
+	5350 1950 5800 1950
 Wire Wire Line
 	6100 1950 6250 1950
@@
 	3350 3650 3200 3650
 Wire Wire Line
-	3200 3650 3200 3750
-Wire Wire Line
-	3200 3750 3200 4000
+	3200 3650 3200 4000
 Wire Wire Line
 	3350 3750 3200 3750
@@
 Wire Notes Line
 	5000 3200 3000 3200
+Text Notes 3750 3300 0    39   ~ 0
+Cortex Debugger
 $EndSCHEMATC

Commit message: Updated to KiCad 5
Parts:
- C201, C202: symbol C_Small -> Device:C_Small
- C203: renamed from C201; symbol C -> Device:C
- C204: renamed from C202; symbol C -> Device:C
- D201: symbol PRTR5V0U2X -> prtr5v0u2x:PRTR5V0U2X
- F201: renamed from F?; symbol Polyfuse -> Device:Polyfuse
- J201: symbol Conn_01x06 -> conn:Conn_01x06
- J202: renamed from J?; symbol Cortex_Debug -> cortex_debug:Cortex_Debug
- J203: renamed from J1; symbol Conn_01x04 -> conn:Conn_01x04
- J204: renamed from J2; symbol Conn_01x06 -> conn:Conn_01x06
- L201: symbol Ferrite_Bead -> Device:Ferrite_Bead
- R201, R202, R203, R204: symbol R -> Device:R
- SW1, SW2: symbol SW_Push -> switches:SW_Push
Connections:
- no-connect marks 1 -> 6
Changed lines of the file:
@@
-EESchema Schematic File Version 2
-LIBS:power
-LIBS:device
-LIBS:switches
-LIBS:relays
-LIBS:motors
-LIBS:transistors
-LIBS:conn
-LIBS:linear
-LIBS:regul
-LIBS:74xx
-LIBS:cmos4000
-LIBS:adc-dac
-LIBS:memory
-LIBS:xilinx
-LIBS:microcontrollers
-LIBS:dsp
-LIBS:microchip
-LIBS:analog_switches
-LIBS:motorola
-LIBS:texas
-LIBS:intel
-LIBS:audio
-LIBS:interface
-LIBS:digital-audio
-LIBS:philips
-LIBS:display
-LIBS:cypress
-LIBS:siliconi
-LIBS:opto
-LIBS:atmel
-LIBS:contrib
-LIBS:valves
-LIBS:TI_Additions
-LIBS:KingBright_Addition
-LIBS:lm2734
-LIBS:prtr5v0u2x
-LIBS:samd21g18a-au
-LIBS:zldo1117-5v
-LIBS:cortex_debug
+EESchema Schematic File Version 4
 LIBS:FSAE Main Panel-cache
-EELAYER 25 0
+EELAYER 26 0
 EELAYER END
 $Descr A4 11693 8268
@@
 $EndDescr
 $Comp
-L Conn_01x04 J1
+L conn:Conn_01x04 J203
 U 1 1 5BE242F9
 P 1050 1250
-F 0 "J1" H 1050 1450 50  0000 C CNN
+F 0 "J203" H 1050 1450 50  0000 C CNN
 F 1 "Conn_01x04" H 1050 950 50  0000 C CNN
 F 2 "" H 1050 1250 50  0001 C CNN
@@
 CAN_V+
 $Comp
-L GND #PWR203
+L power:GND #PWR204
 U 1 1 5BE24FFA
 P 1900 1450
-F 0 "#PWR203" H 1900 1200 50  0001 C CNN
+F 0 "#PWR204" H 1900 1200 50  0001 C CNN
 F 1 "GND" V 1900 1250 50  0000 C CNN
 F 2 "" H 1900 1450 50  0001 C CNN
@@
 CAN_L
 $Comp
-L Conn_01x06 J2
+L conn:Conn_01x06 J204
 U 1 1 5BE9B0A3
 P 1050 2250
-F 0 "J2" H 1050 2550 50  0000 C CNN
+F 0 "J204" H 1050 2550 50  0000 C CNN
 F 1 "TE_84953-6_FPC" H 1050 1850 50  0000 C CNN
 F 2 "Connectors_TE-Connectivity:TE_84953-6_1x06_P1.0mm_Horizontal" H 1050 2250 50  0001 C CNN
@@
 DWC_+5V
 $Comp
-L GND #PWR204
+L power:GND #PWR203
 U 1 1 5BE9B884
 P 1850 2150
-F 0 "#PWR204" H 1850 1900 50  0001 C CNN
+F 0 "#PWR203" H 1850 1900 50  0001 C CNN
 F 1 "GND" V 1850 1950 50  0000 C CNN
 F 2 "" H 1850 2150 50  0001 C CNN
@@
 Dashboard Warning Light Cluster
 $Comp
-L SW_Push SW1
+L switches:SW_Push SW1
 U 1 1 5BE9B978
 P 1000 3250
@@
 MCU Reset
 $Comp
-L SW_Push SW2
+L switches:SW_Push SW2
 U 1 1 5BE9BA9C
 P 1000 4150
@@
 Alarm Clear
 $Comp
-L GND #PWR201
+L power:GND #PWR201
 U 1 1 5BE9BAFE
 P 750 3400
@@
 $EndComp
 $Comp
-L GND #PWR202
+L power:GND #PWR202
 U 1 1 5BE9BB22
 P 750 4300
@@
 $EndComp
 $Comp
-L R R201
+L Device:R R201
 U 1 1 5BE9BDD1
 P 1950 3250
@@
 ~RESET
 $Comp
-L C_Small C201
+L Device:C_Small C201
 U 1 1 5BE9C881
 P 1950 3050
@@
 $EndComp
 $Comp
-L R R202
+L Device:R R202
 U 1 1 5BE9C8E2
 P 1450 3250
@@
 $EndComp
 $Comp
-L R R203
+L Device:R R203
 U 1 1 5BE9CBCA
 P 1950 4150
@@
 ~CLEAR
 $Comp
-L C_Small C202
+L Device:C_Small C202
 U 1 1 5BE9CBDF
 P 1950 3950
@@
 $EndComp
 $Comp
-L R R204
+L Device:R R204
 U 1 1 5BE9CBE5
 P 1450 4150
@@
 $EndComp
 $Comp
-L +3.3V #PWR205
+L power:+3.3V #PWR205
 U 1 1 5BE9CCF2
 P 2300 3250
@@
 $EndComp
 $Comp
-L +3.3V #PWR206
+L power:+3.3V #PWR206
 U 1 1 5BE9CD22
 P 2300 4150
@@
 $EndComp
 $Comp
-L Conn_01x06 J201
+L conn:Conn_01x06 J201
 U 1 1 5BF06479
 P 3200 2150
-F 0 "J201" H 3200 2350 50  0000 C CNN
+F 0 "J201" H 3200 2450 50  0000 C CNN
 F 1 "Conn_01x06" V 3300 2100 50  0000 C CNN
 F 2 "" H 3200 2150 50  0001 C CNN
@@
 $EndComp
 $Comp
-L GND #PWR207
+L power:GND #PWR209
 U 1 1 5BF06480
 P 4000 2800
-F 0 "#PWR207" H 4000 2550 50  0001 C CNN
+F 0 "#PWR209" H 4000 2550 50  0001 C CNN
 F 1 "GND" H 4000 2650 50  0000 C CNN
 F 2 "" H 4000 2800 50  0001 C CNN
@@
 $EndComp
 $Comp
-L Ferrite_Bead L201
+L Device:Ferrite_Bead L201
 U 1 1 5BF06486
 P 5200 1950
@@
 $EndComp
 $Comp
-L C C201
+L Device:C C203
 U 1 1 5BF06494
 P 4450 2500
-F 0 "C201" H 4475 2600 50  0000 L CNN
+F 0 "C203" H 4475 2600 50  0000 L CNN
 F 1 "4.7nF" H 4475 2400 50  0000 L CNN
 F 2 "" H 4488 2350 50  0001 C CNN
@@
 $EndComp
 $Comp
-L PRTR5V0U2X D201
+L prtr5v0u2x:PRTR5V0U2X D201
 U 1 1 5BF064A8
 P 4300 1400
@@
 USB_POWER
 $Comp
-L C C202
+L Device:C C204
 U 1 1 5BF0649B
 P 5600 2500
-F 0 "C202" H 5625 2600 50  0000 L CNN
+F 0 "C204" H 5625 2600 50  0000 L CNN
 F 1 "4.7nF" H 5625 2400 50  0000 L CNN
 F 2 "" H 5638 2350 50  0001 C CNN
@@
 	4800 1200 4900 1200
 Wire Wire Line
-	4900 2750 4900 1200
+	4900 1200 4900 2750
 Wire Wire Line
 	5600 2750 5600 2650
@@
 	650  850  650  1650
 $Comp
-L Polyfuse F?
+L Device:Polyfuse F201
 U 1 1 5BF9A374
 P 5950 1950
-F 0 "F?" V 5850 1950 50  0000 C CNN
+F 0 "F201" V 5850 1950 50  0000 C CNN
 F 1 "MF-MSMF050-2" V 5750 1950 50  0000 C CNN
 F 2 "" H 6000 1750 50  0001 L CNN
@@
 	6100 1950 6250 1950
 $Comp
-L Cortex_Debug J?
+L cortex_debug:Cortex_Debug J202
 U 1 1 5BFE970B
 P 3950 3750
-F 0 "J?" H 3950 4050 50  0000 C CNN
+F 0 "J202" H 3950 4050 50  0000 C CNN
 F 1 "Cortex_Debug" H 3950 3450 50  0000 C CNN
 F 2 "" H 4100 3750 39  0001 C CNN
@@
 $EndComp
 $Comp
-L +3.3V #PWR?
+L power:+3.3V #PWR207
 U 1 1 5BFE98A3
 P 3200 3400
-F 0 "#PWR?" H 3200 3250 50  0001 C CNN
+F 0 "#PWR207" H 3200 3250 50  0001 C CNN
 F 1 "+3.3V" H 3200 3540 50  0000 C CNN
 F 2 "" H 3200 3400 50  0001 C CNN
@@
 $EndComp
 $Comp
-L GND #PWR?
+L power:GND #PWR208
 U 1 1 5BFE993E
 P 3200 4000
-F 0 "#PWR?" H 3200 3750 50  0001 C CNN
+F 0 "#PWR208" H 3200 3750 50  0001 C CNN
 F 1 "GND" H 3200 3850 50  0000 C CNN
 F 2 "" H 3200 4000 50  0001 C CNN
@@
 Text Notes 3750 3300 0    39   ~ 0
 Cortex Debugger
+NoConn ~ 4550 3750
+NoConn ~ 4550 3850
+NoConn ~ 4550 3950
+NoConn ~ 3350 3850
+NoConn ~ 3350 3950
 $EndSCHEMATC
